Commit message: Rename ackmann to ackermann and update simulation/nav configs

File: src/robot_description/urdf/diff_sensors.urdf (robot description, URDF)
Before this commit: robot diff_robot, 9 links, 8 joints
Links:
- link $(arg ns)/base_link: geometry collision box size=0.2 0.1 0.01; collision sphere radius=0.01
- link $(arg ns)/camera_frame: geometry visual mesh filename=package://description_robot/models/diffbot/meshes/d435.dae scale=1.0 1.0 1.0
- link $(arg ns)/caster_base_link: geometry visual mesh filename=package://description_robot/models/diffbot/meshes/base_cast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
- link $(arg ns)/caster_wheel_link: geometry collision cylinder length=0.01 radius=0.015; visual mesh filename=package://description_robot/models/diffbot/meshes/caster_wh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
- link $(arg ns)/lidar_link: geometry visual mesh filename=package://description_robot/models/diffbot/meshes/Lidar_pac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 scale=0.001 0.001 0.001
- link $(arg ns)/rgbd_camera_frame: geometry visual mesh filename=package://description_robot/models/diffbot/meshes/d435.dae scale=1.0 1.0 1.0
- link $(arg ns)/wheel_left_link: geometry collision cylinder length=${wheelThickness} radius=${wheelDiameter/2}; visual mesh filename=package://description_robot/models/diffbot/meshes/wheel_rin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 scale=1 1 1
- link $(arg ns)/wheel_right_link: geometry collision cylinder length=${wheelThickness} radius=${wheelDiameter/2}; visual mesh filename=package://description_robot/models/diffbot/meshes/wheel_rin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 scale=1 1 1

File: src/robot_description/urdf/donkey_sensors.urdf (robot description, URDF)
Before this commit: robot ackmann, 8 links, 7 joints
Links:
- link $(arg ns)/base_link: geometry collision box size=.3 .09 .12; visual mesh filename=package://description_robot/models/donkey/meshes/BaseReduce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 scale=1 1 1
- link $(arg ns)/front_left_wheel_link: geometry collision cylinder length=0.03 radius=0.0365; visual mesh filename=package://description_robot/models/donkey/meshes/Wheel.dae
- link $(arg ns)/front_right_wheel_link: geometry collision cylinder length=0.03 radius=0.0365; visual mesh filename=package://description_robot/models/donkey/meshes/Wheel.dae
- link $(arg ns)/rear_left_wheel_link: geometry collision cylinder length=0.03 radius=0.0365; visual mesh filename=package://description_robot/models/donkey/meshes/Wheel.dae
- link $(arg ns)/rear_right_wheel_link: geometry collision cylinder length=0.03 radius=0.0365; visual mesh filename=package://description_robot/models/donkey/meshes/Wheel.dae

File: src/robot_description/urdf/realsense/_l515.urdf.xacro (robot description, xacro)
@@ -63,5 +63,5 @@
           <origin xyz="${l515_zero_depth_to_glass} 0 ${-l515_cam_center_to_depth_pz}" rpy="${M_PI/2} 0 ${M_PI/2}"/>
           <geometry>
-              <mesh filename="package://robot_description/urdf/realsense/meshes/l515.dae" />
+	      <mesh filename="package://description_robot/urdf/realsense/meshes/l515.dae" />
           </geometry>
         </xacro:if>

File: src/robot_description/urdf/sensors/rplidar.urdf.xacro (robot description, xacro)
@@ -2,5 +2,5 @@
 <robot xmlns:xacro="http://ros.org/wiki/xacro">
 <xacro:macro name="rplidar" params="name parent_link gazebo *origin">
-  <xacro:include filename="$(find robot_description)/urdf/common_properties.urdf.xacro"/>
+  <xacro:include filename="$(find description_robot)/urdf/common_properties.urdf.xacro"/>
   <xacro:property name="mass"       value="0.17"/>
   <xacro:property name="length_x"   value="${7.1*cm2m}" />
