Commit message: update urdf, tf still not fixed

File: src/description_robot/urdf/common_properties.urdf.xacro (robot description, xacro)
@@ -86,4 +86,5 @@
       <sensor name="${sensor_name}" type="gpu_lidar">
         <update_rate>${update_rate}</update_rate>
+        <ignition_frame_id>${sensor_name}_link</ignition_frame_id>
         <topic>/rplidar/scan</topic>
         <visualize>${visualize}</visualize>

File: src/description_robot/urdf/realsense/_d435i.urdf.xacro (robot description, xacro)
@@ -8,10 +8,14 @@
 <robot name="sensor_d435i" xmlns:xacro="http://ros.org/wiki/xacro">
   <xacro:include filename="$(find realsense2_description)/urdf/_d435.urdf.xacro"/>
-  <xacro:include filename="$(find realsense2_description)/urdf/_d435i_imu_modules.urdf.xacro"/>
-  <xacro:macro name="sensor_d435i" params="parent *origin name:=camera use_nominal_extrinsics:=false">
+  <xacro:include filename="$(find description_robot)/urdf/realsense/_d435i_imu_modules.urdf.xacro"/>
+  <xacro:include filename="$(find description_robot)/urdf/realsense/_d435i_sensors.urdf.xacro"/>
+  <xacro:macro name="sensor_d435i" params="parent *origin name:=camera use_nominal_extrinsics:=false add_plug:=false use_mesh:=true add_sensors:=true">
     <xacro:sensor_d435 parent="${parent}" name="${name}" use_nominal_extrinsics="${use_nominal_extrinsics}">
       <xacro:insert_block name="origin" />
     </xacro:sensor_d435>
     <xacro:d435i_imu_modules name="${name}" use_nominal_extrinsics="${use_nominal_extrinsics}"/>
+    <xacro:if value="${add_sensors}">
+      <xacro:gazebo_d435i parent="${parent}" name="${name}" width="640" height="480" fov="1.39626" image_fps="30" accel_fps="62.5" gyro_fps="200"/>
+    </xacro:if>
   </xacro:macro>
 </robot>

File: src/description_robot/urdf/realsense/_l515.urdf.xacro (robot description, xacro)
@@ -10,5 +10,6 @@
   <xacro:include filename="$(find realsense2_description)/urdf/_materials.urdf.xacro" />
   <xacro:include filename="$(find realsense2_description)/urdf/_usb_plug.urdf.xacro" /> <!-- this specific plug does not apply to L515 -->
-  <xacro:macro name="sensor_l515" params="parent *origin name:=camera use_nominal_extrinsics:=false add_plug:=false use_mesh:=true">
+  <xacro:include filename="$(find description_robot)/urdf/realsense/_l515_sensors.urdf.xacro"/>
+  <xacro:macro name="sensor_l515" params="parent *origin name:=camera use_nominal_extrinsics:=false add_plug:=false use_mesh:=true add_sensors:=true">
     <xacro:property name="M_PI" value="3.1415926535897931" />
     <!-- The following values are approximate, and the camera node
@@ -63,5 +64,5 @@
           <origin xyz="${l515_zero_depth_to_glass} 0 ${-l515_cam_center_to_depth_pz}" rpy="${M_PI/2} 0 ${M_PI/2}"/>
           <geometry>
-	      <mesh filename="package://description_robot/urdf/realsense/meshes/l515.dae" />
+              <mesh filename="package://description_robot/urdf/realsense/meshes/l515.dae" />
           </geometry>
         </xacro:if>
@@ -177,4 +178,7 @@
       </xacro:usb_plug>
     </xacro:if>
+    <xacro:if value="${add_sensors}">
+      <xacro:gazebo_l515 parent="${parent}" name="${name}" width="640" height="480" fov="1.39626" image_fps="30" accel_fps="62.5" gyro_fps="200"/>
+    </xacro:if>
   </xacro:macro>
 </robot>

File: src/description_robot/urdf/sensors/rplidar.urdf.xacro (robot description, xacro)
@@ -15,11 +15,13 @@
     <xacro:insert_block name="origin"/>
   </joint>
-  <link name="${name}_link">
+    <link name="${name}_link">
     <visual>
       <origin xyz="0 0 0" rpy="0 0 0"/>
       <geometry>
-        <cylinder radius="0.04" length="0.07"/>
+        <cylinder radius="0.03" length="0.02" />
       </geometry>
-      <material name="dark_gray"/>
+      <material name="dark_gray">
+        <color rgba="0.2 0.2 0.2 1.0"/>
+      </material>
     </visual>
     <collision>

Commit message: update model file for gazebo harmonic to fix tf frame issue

File: src/description_robot/urdf/common_properties.urdf.xacro (robot description, xacro)
@@ -87,4 +87,5 @@
         <update_rate>${update_rate}</update_rate>
         <ignition_frame_id>${sensor_name}_link</ignition_frame_id>
+        <gz_frame_id>${sensor_name}_link</gz_frame_id>
         <topic>/rplidar/scan</topic>
         <visualize>${visualize}</visualize>
@@ -113,5 +114,5 @@
       </sensor>
     </xacro:if>
-  </xacro:macro>
+    </xacro:macro>
   <!-- Conversion macros -->
   <xacro:property name="cm2m"    value="${1/100.0}"/>

File: src/description_robot/urdf/realsense/_d435i_sensors.urdf.xacro (robot description, xacro)
@@ -95,4 +95,5 @@
         <topic>/${name}/imu</topic>
         <ignition_frame_id>${name}_imu_optical_frame</ignition_frame_id>
+        <gz_frame_id>${name}_imu_optical_frame</gz_frame_id>
         <imu>
           <angular_velocity>

File: src/description_robot/urdf/realsense/_l515_sensors.urdf.xacro (robot description, xacro)
@@ -67,4 +67,5 @@
       <visualize>false</visualize>
       <topic>/${name}/imu/raw</topic>
+      <ignition_frame_id>${name}_imu_optical_frame</ignition_frame_id>
       <gz_frame_id>${name}_imu_optical_frame</gz_frame_id>
       <imu>

File: src/description_robot/urdf/realsense/_t265_sensors.urdf.xacro (robot description, xacro)
@@ -105,4 +105,5 @@
         <topic>/${name}/imu</topic>
         <ignition_frame_id>${name}_imu_optical_frame</ignition_frame_id>
+        <gz_frame_id>${name}_imu_optical_frame</gz_frame_id>
         <imu>
           <angular_velocity>
