Commit message: udpate urdf

File: src/description_robot/urdf/diff_sensors.urdf (robot description, URDF)
Before this commit: robot diff_robot, 9 links, 8 joints
Joints:
- joint $(arg ns)/base_joint: child $(arg ns)/base_link -> $(arg ns)/base_footprint; origin xyz=0 0 ${base_elevation} rpy=0 0 0 -> xyz=0 0 ${-base_elevation} rpy=0 0 0; parent $(arg ns)/base_footprint -> $(arg ns)/base_link

File: src/description_robot/urdf/donkey_sensors.urdf (robot description, URDF)
Before this commit: robot ackermann, 8 links, 7 joints
Joints:
- joint $(arg ns)/base_joint: child $(arg ns)/base_link -> $(arg ns)/base_footprint; origin xyz=0 0 ${base_elevation} rpy=0 0 0 -> xyz=0 0 ${-base_elevation} rpy=0 0 0; parent $(arg ns)/base_footprint -> $(arg ns)/base_link
