Commit message: fix: move base_link origin to rear axle centre, keep same z
Shift base_link from mid-wheelbase to the rear axle midpoint
(+wheel_base/2 = +0.087 m in X). All child positions updated
to keep every component at the same world location:

- Rear wheel joints: x = 0 (was -wheel_base/2)
- Front steering joints: x = wheel_base (was wheel_base/2)
- Body visual/collision/inertial: x += wheel_base/2
- All sensor x offsets (d435i, t265, l515, rplidar, cubepilot):
  expressed as original_offset + wheel_base/2

Co-Authored-By: Claude Opus 4.6 <noreply@anthropic.com>

File: src/description_robot/urdf/donkey_sensors.urdf (robot description, URDF)
Before this commit: robot ackermann, 8 links, 7 joints
Joints:
- joint $(arg ns)/front_left_wheel_steering_joint: origin xyz=${wheel_base/2} ${wheel_separation/2} 0 rpy=0 0 0 -> xyz=${wheel_base} ${wheel_separation/2} 0 rpy=0 0 0
- joint $(arg ns)/front_right_wheel_steering_joint: origin xyz=${wheel_base/2} ${-wheel_separation/2} 0 rpy=0 0 0 -> xyz=${wheel_base} ${-wheel_separation/2} 0 rpy=0 0 0
- joint $(arg ns)/rear_left_wheel_joint: origin xyz=${-wheel_base/2} ${wheel_separation/2} 0 rpy=0 0 0 -> xyz=0 ${wheel_separation/2} 0 rpy=0 0 0
- joint $(arg ns)/rear_right_wheel_joint: origin xyz=${-wheel_base/2} ${-wheel_separation/2} 0 rpy=0 0 0 -> xyz=0 ${-wheel_separation/2} 0 rpy=0 0 0
