Commit message: feat: add CubePilot xacro with mount_link and IMU sensor, fix T265 frame offsets
- Add cubepilot.urdf.xacro with mount_link -> cubepilot_link (geometric centre)
  -> cubepilot_imu_link chain, Gazebo IMU sensor plugin, and STL mesh
- Add cubepilot.stl mesh for Gazebo visualization
- Include cubepilot macro in donkey_sensors.urdf with offset properties
- Add /cubepilot/imu bridge topic to gazebo_bringup.launch.py
- Fix T265 pose_joint: remove duplicate origin block, add correct 21mm Y offset
- Fix T265 accel/gyro joints: correct offset from 210mm to 21mm in +Y
- Remove non-ASCII characters (degree signs, arrows) from all xacro/urdf
  comments to prevent YAML parse failures in robot_description parameter

File: src/description_robot/urdf/realsense/_t265.urdf.xacro (robot description, xacro)
@@ -30,5 +30,5 @@
     <!-- camera body, with origin at camera_pose_frame -->
     <joint name="${name}_pose_joint" type="fixed">
-      <xacro:insert_block name="origin"/>
+      <origin xyz="0 0.021 0" rpy="0 0 0"/>
       <parent link="${name}_link"/>
       <child link="${name}_pose_frame"/>
@@ -81,5 +81,5 @@
     <!-- IMU joints and links -->
     <joint name="${name}_accel_joint" type="fixed">
-      <origin xyz="0 0.21 0" rpy="0 0 ${M_PI}"/>
+      <origin xyz="0 0.021 0" rpy="0 0 ${M_PI}"/>
       <parent link="${name}_link"/>
       <child link="${name}_accel_frame"/>
@@ -93,5 +93,5 @@
     <link name="${name}_accel_optical_frame"/>
     <joint name="${name}_gyro_joint" type="fixed">
-      <origin xyz="0 0.21 0" rpy="0 0 ${M_PI}"/>
+      <origin xyz="0 0.021 0" rpy="0 0 ${M_PI}"/>
       <parent link="${name}_link"/>
       <child link="${name}_gyro_frame"/>

File: src/description_robot/urdf/realsense/_t265_sensors.urdf.xacro (robot description, xacro)
@@ -33,5 +33,5 @@
           <type>equisolid_angle</type>
           <scale_to_hfov>true</scale_to_hfov>
-          <cutoff_angle>${fov/2}</cutoff_angle>  <!-- 85° cutoff -->
+          <cutoff_angle>${fov/2}</cutoff_angle>  <!-- 85 deg cutoff -->
           <env_texture_size>1024</env_texture_size>
           <!-- <intrinsics>
@@ -79,5 +79,5 @@
           <type>equisolid_angle</type>
           <scale_to_hfov>true</scale_to_hfov>
-          <cutoff_angle>${fov/2}</cutoff_angle>  <!-- 85° cutoff -->
+          <cutoff_angle>${fov/2}</cutoff_angle>  <!-- 85 deg cutoff -->
           <env_texture_size>1024</env_texture_size>
           <!-- <intrinsics>
