Commit message: fix: correct T265 URDF frame hierarchy and Gazebo odometry plugin
- Move mesh/collision/inertial from camera_pose_frame to camera_link
  (the physical body is camera_link, not the pose frame)
- Define camera_pose_frame as a static identity child of camera_link;
  driver must run with publish_tf:=false to avoid TF conflicts
- Fix camera_pose_joint to use identity transform (was incorrectly
  re-applying the mount origin, double-offsetting the pose frame)
- Fix IMU accel/gyro joint offset from 0.21m to 0.021m
- Change Gazebo OdometryPublisher robot_base_frame from
  camera_pose_frame to camera_link so Gazebo tracks the physical
  body; EKF consumes the odometry and owns odom_frame->base_link TF

Co-Authored-By: Claude Opus 4.6 <noreply@anthropic.com>

File: src/description_robot/urdf/realsense/_t265.urdf.xacro (robot description, xacro)
@@ -22,19 +22,11 @@
     <!-- camera body, with origin at camera_link -->
     <joint name="${name}_link_joint" type="fixed">
-      <!-- <origin xyz="0 0 0" rpy="0 0 0"/> -->
       <xacro:insert_block name="origin"/>
       <parent link="${parent}"/>
       <child link="${name}_link"/>
     </joint>
-    <link name="${name}_link"/>
-    <!-- camera body, with origin at camera_pose_frame -->
-    <joint name="${name}_pose_joint" type="fixed">
-      <origin xyz="0 0.021 0" rpy="0 0 0"/>
-      <parent link="${name}_link"/>
-      <child link="${name}_pose_frame"/>
-    </joint>
-    <link name="${name}_pose_frame">
+    <link name="${name}_link">
       <visual>
-      <origin xyz="0 0 0" rpy="${M_PI / 2} 0 ${M_PI /2}"/>
+        <origin xyz="0 0 0" rpy="${M_PI / 2} 0 ${M_PI /2}"/>
         <geometry>
             <mesh filename="package://description_robot/urdf/realsense/meshes/t265.stl" scale="0.001 0.001 0.001"/>
@@ -55,4 +47,14 @@
       </inertial>
     </link>
+    <!-- camera_pose_frame is a static identity child of camera_link.
+         The T265 driver must be configured with publish_tf:=false so it does
+         not publish competing TF for this frame. Only odometry data is consumed
+         (fed to an EKF which owns the odom_frame -> base_link edge). -->
+    <joint name="${name}_pose_joint" type="fixed">
+      <origin xyz="0 0 0" rpy="0 0 0"/>
+      <parent link="${name}_link"/>
+      <child link="${name}_pose_frame"/>
+    </joint>
+    <link name="${name}_pose_frame"/>
     <joint name="${name}_fisheye1_joint" type="fixed">
       <origin xyz="${fisheye1_offset_x} ${fisheye1_offset_y} ${fisheye1_offset_z}" rpy="${-M_PI} 0 ${-M_PI}"/>

File: src/description_robot/urdf/realsense/_t265_sensors.urdf.xacro (robot description, xacro)
@@ -126,5 +126,5 @@
         <dimensions>3</dimensions>
         <odom_frame>odom_frame</odom_frame>
-        <robot_base_frame>${name}_pose_frame</robot_base_frame>
+        <robot_base_frame>${name}_link</robot_base_frame>
         <publish_link_pose>true</publish_link_pose>
         <tf_topic>$(arg ns)/tf</tf_topic>
