Commit message: refactor: move URDF to models/ackermann_rover, fix robot motion
- Move urdf/ to models/ackermann_rover/, rename donkey_sensors.urdf to ackermann_rover.urdf
- Update all launch files and xacro includes for new paths
- Fix robot not moving: wrap PX4 SITL joint plugins in enable_px4_sitl conditional
- Set reference_timeout to 0.0 in ackermann_controller.yaml
- Add enable_px4_sitl launch arg to gazebo_bringup.launch.py
- Add verification log and motion test script
- Add stop command docs to README

File: src/description_robot/models/ackermann_rover/cubepilot/cubepilot.urdf.xacro (robot description, xacro)
@@ -12,5 +12,5 @@
 -->
 <robot xmlns:xacro="http://ros.org/wiki/xacro">
-  <xacro:include filename="$(find description_robot)/urdf/common_properties.urdf.xacro"/>
+  <xacro:include filename="$(find description_robot)/models/ackermann_rover/common_properties.urdf.xacro"/>
   <xacro:macro name="cubepilot" params="name parent_link *origin
                                          imu_update_rate:=200
@@ -37,5 +37,5 @@
         <origin xyz="0 0 0" rpy="0 0 0"/>
         <geometry>
-          <mesh filename="package://description_robot/urdf/cubepilot/cubepilot.stl" scale="0.001 0.001 0.001"/>
+          <mesh filename="package://description_robot/models/ackermann_rover/cubepilot/cubepilot.stl" scale="0.001 0.001 0.001"/>
         </geometry>
         <material name="cubepilot_gray">

File: src/description_robot/models/ackermann_rover/realsense/_d435i.urdf.xacro (robot description, xacro)
@@ -8,6 +8,6 @@
 <robot name="sensor_d435i" xmlns:xacro="http://ros.org/wiki/xacro">
   <xacro:include filename="$(find realsense2_description)/urdf/_d435.urdf.xacro"/>
-  <xacro:include filename="$(find description_robot)/urdf/realsense/_d435i_imu_modules.urdf.xacro"/>
-  <xacro:include filename="$(find description_robot)/urdf/realsense/_d435i_sensors.urdf.xacro"/>
+  <xacro:include filename="$(find description_robot)/models/ackermann_rover/realsense/_d435i_imu_modules.urdf.xacro"/>
+  <xacro:include filename="$(find description_robot)/models/ackermann_rover/realsense/_d435i_sensors.urdf.xacro"/>
   <xacro:macro name="sensor_d435i" params="parent *origin name:=camera use_nominal_extrinsics:=false add_plug:=false use_mesh:=true add_sensors:=true">
     <xacro:sensor_d435 parent="${parent}" name="${name}" use_nominal_extrinsics="${use_nominal_extrinsics}">

File: src/description_robot/models/ackermann_rover/realsense/_l515.urdf.xacro (robot description, xacro)
@@ -10,5 +10,5 @@
   <xacro:include filename="$(find realsense2_description)/urdf/_materials.urdf.xacro" />
   <xacro:include filename="$(find realsense2_description)/urdf/_usb_plug.urdf.xacro" /> <!-- this specific plug does not apply to L515 -->
-  <xacro:include filename="$(find description_robot)/urdf/realsense/_l515_sensors.urdf.xacro"/>
+  <xacro:include filename="$(find description_robot)/models/ackermann_rover/realsense/_l515_sensors.urdf.xacro"/>
   <xacro:macro name="sensor_l515" params="parent *origin name:=camera use_nominal_extrinsics:=false add_plug:=false use_mesh:=true add_sensors:=true">
     <xacro:property name="M_PI" value="3.1415926535897931" />
@@ -64,5 +64,5 @@
           <origin xyz="${l515_zero_depth_to_glass} 0 ${-l515_cam_center_to_depth_pz}" rpy="${M_PI/2} 0 ${M_PI/2}"/>
           <geometry>
-              <mesh filename="package://description_robot/urdf/realsense/meshes/l515.dae" />
+              <mesh filename="package://description_robot/models/ackermann_rover/realsense/meshes/l515.dae" />
           </geometry>
         </xacro:if>

File: src/description_robot/models/ackermann_rover/realsense/_t265.urdf.xacro (robot description, xacro)
@@ -2,5 +2,5 @@
 <robot name="sensor_t265" xmlns:xacro="http://ros.org/wiki/xacro">
   <!-- includes-->
-  <xacro:include filename="$(find description_robot)/urdf/realsense/_t265_sensors.urdf.xacro"/>
+  <xacro:include filename="$(find description_robot)/models/ackermann_rover/realsense/_t265_sensors.urdf.xacro"/>
     <!-- odom_xyz, odom_rpy params are the transformation from the robot base_link to the camera reference frame (camerea_pose_frame)
   they are needed for the simulation of the camera slam capabilities -->
@@ -30,5 +30,5 @@
         <origin xyz="0 0 0" rpy="${M_PI / 2} 0 ${M_PI /2}"/>
         <geometry>
-            <mesh filename="package://description_robot/urdf/realsense/meshes/t265.stl" scale="0.001 0.001 0.001"/>
+            <mesh filename="package://description_robot/models/ackermann_rover/realsense/meshes/t265.stl" scale="0.001 0.001 0.001"/>
         </geometry>
         <material name="${name}_aluminum"/>
@@ -37,5 +37,5 @@
         <origin xyz="0 0 0" rpy="${M_PI / 2} 0 ${M_PI /2}"/>
         <geometry>
-          <mesh filename="package://description_robot/urdf/realsense/meshes/t265.stl"  scale="0.001 0.001 0.001"/>
+          <mesh filename="package://description_robot/models/ackermann_rover/realsense/meshes/t265.stl"  scale="0.001 0.001 0.001"/>
         </geometry>
       </collision>

File: src/description_robot/models/ackermann_rover/sensors/rplidar.urdf.xacro (robot description, xacro)
@@ -2,5 +2,5 @@
 <robot xmlns:xacro="http://ros.org/wiki/xacro">
 <xacro:macro name="rplidar" params="name parent_link gazebo *origin">
-  <xacro:include filename="$(find description_robot)/urdf/common_properties.urdf.xacro"/>
+  <xacro:include filename="$(find description_robot)/models/ackermann_rover/common_properties.urdf.xacro"/>
   <xacro:property name="mass"       value="0.17"/>
   <xacro:property name="length_x"   value="${7.1*cm2m}" />

Commit message: feat: PX4 SITL co-simulation integration
- Add PX4 build dependencies to Docker image
- Create px4_requirements.txt for PX4 Python build deps
- Change PX4 mount from :ro to read-write in docker-compose
- Add enable_px4_sitl mode to cubepilot.urdf.xacro with PX4-compatible
  base_link sensors (imu, baro, mag, navsat)
- Pass enable_px4_sitl arg through ackermann_rover.urdf and launch files
- Add spherical_coordinates to warehouse.sdf (Zurich reference)
- Skip ros2_control spawn when PX4 mode in gazebo_bringup.launch.py
- Add start_px4_sitl.sh and stop_all.sh scripts
- Document full PX4 SITL verification (16/16 checkpoints pass)

File: src/description_robot/models/ackermann_rover/cubepilot/cubepilot.urdf.xacro (robot description, xacro)
@@ -10,8 +10,12 @@
   Internal IMU offset from board center: approximately 6 mm forward, 6 mm right, 4 mm down
   (see CubeOrange IMU1 datasheet for exact values).
+  When enable_px4_sitl is true, an additional "base_link" (no namespace prefix) is
+  created with PX4-compatible sensor names so that PX4 gz_bridge can discover them
+  at its hardcoded topic paths: /world/{world}/model/{model}/link/base_link/sensor/{name}/{type}
 -->
 <robot xmlns:xacro="http://ros.org/wiki/xacro">
   <xacro:include filename="$(find description_robot)/models/ackermann_rover/common_properties.urdf.xacro"/>
   <xacro:macro name="cubepilot" params="name parent_link *origin
+                                         enable_px4_sitl:=false
                                          imu_update_rate:=200
                                          imu_topic:=/cubepilot/imu
@@ -51,5 +55,6 @@
       <xacro:inertial_cuboid mass="${board_mass}" x="${board_x}" y="${board_y}" z="${board_z}"/>
     </link>
-    <!-- =============== All Gazebo sensors on single link =============== -->
+    <!-- =============== Gazebo sensors (standard mode) =============== -->
+    <xacro:unless value="${enable_px4_sitl}">
     <gazebo reference="${name}_link">
       <!-- IMU -->
@@ -109,4 +114,73 @@
       <xacro:material_darkgray/>
     </gazebo>
+    </xacro:unless>
+    <!-- =============== PX4 SITL sensors on "base_link" =============== -->
+    <!-- PX4 gz_bridge hardcodes: /world/{w}/model/{m}/link/base_link/sensor/{name}/{type}
+         We create a separate link named exactly "base_link" (no namespace) so
+         the Gazebo topic path matches PX4's expectation. -->
+    <xacro:if value="${enable_px4_sitl}">
+    <joint name="px4_base_link_joint" type="fixed">
+      <parent link="${parent_link}"/>
+      <child link="base_link"/>
+      <origin xyz="0 0 0" rpy="0 0 0"/>
+    </joint>
+    <link name="base_link">
+      <inertial>
+        <mass value="0.001"/>
+        <inertia ixx="1e-7" ixy="0" ixz="0" iyy="1e-7" iyz="0" izz="1e-7"/>
+      </inertial>
+    </link>
+    <gazebo reference="base_link">
+      <sensor name="imu_sensor" type="imu">
+        <always_on>true</always_on>
+        <update_rate>${imu_update_rate}</update_rate>
+        <visualize>false</visualize>
+        <gz_frame_id>base_link</gz_frame_id>
+        <imu>
+          <angular_velocity>
+            <x><noise type="gaussian"><mean>0.0</mean><stddev>0.0002</stddev></noise></x>
+            <y><noise type="gaussian"><mean>0.0</mean><stddev>0.0002</stddev></noise></y>
+            <z><noise type="gaussian"><mean>0.0</mean><stddev>0.0002</stddev></noise></z>
+          </angular_velocity>
+          <linear_acceleration>
+            <x><noise type="gaussian"><mean>0.0</mean><stddev>0.017</stddev></noise></x>
+            <y><noise type="gaussian"><mean>0.0</mean><stddev>0.017</stddev></noise></y>
+            <z><noise type="gaussian"><mean>0.0</mean><stddev>0.017</stddev></noise></z>
+          </linear_acceleration>
+        </imu>
+      </sensor>
+      <sensor name="air_pressure_sensor" type="air_pressure">
+        <always_on>true</always_on>
+        <update_rate>${baro_update_rate}</update_rate>
+        <gz_frame_id>base_link</gz_frame_id>
+        <air_pressure>
+          <pressure>
+            <noise type="gaussian">
+              <mean>0</mean>
+              <stddev>0.01</stddev>
+            </noise>
+          </pressure>
+        </air_pressure>
+      </sensor>
+      <sensor name="magnetometer_sensor" type="magnetometer">
+        <always_on>true</always_on>
+        <update_rate>${mag_update_rate}</update_rate>
+        <gz_frame_id>base_link</gz_frame_id>
+        <magnetometer>
+          <x><noise type="gaussian"><stddev>0.0001</stddev></noise></x>
+          <y><noise type="gaussian"><stddev>0.0001</stddev></noise></y>
+          <z><noise type="gaussian"><stddev>0.0001</stddev></noise></z>
+        </magnetometer>
+      </sensor>
+      <sensor name="navsat_sensor" type="navsat">
+        <always_on>true</always_on>
+        <update_rate>${gps_update_rate}</update_rate>
+        <gz_frame_id>base_link</gz_frame_id>
+      </sensor>
+    </gazebo>
+    <gazebo reference="px4_base_link_joint">
+      <preserveFixedJoint>true</preserveFixedJoint>
+    </gazebo>
+    </xacro:if>
     <gazebo reference="${name}_joint">
       <preserveFixedJoint>true</preserveFixedJoint>

Commit message: feat: add host-side helper scripts, fix stop_all, simplify cubepilot visual\n\n- Add start_ros2_nodes.sh: single command to launch Gazebo/PX4/bridge/SLAM/Nav2\n- Add test_actuators.sh: host-side wrapper for PX4 actuator_test\n- Fix stop_all.sh: include MicroXRCE in pkill pattern to prevent port conflicts\n- Replace cubepilot STL mesh with simple box geometry\n- Update overview.md: quick-start section, actuator test docs with script usage"

File: src/description_robot/models/ackermann_rover/cubepilot/cubepilot.urdf.xacro (robot description, xacro)
@@ -39,7 +39,8 @@
     <link name="${name}_link">
       <visual>
-        <origin xyz="0 0 0" rpy="0 0 0"/>
+        <origin xyz="0 0 ${board_z/2}" rpy="0 0 0"/>
         <geometry>
           <mesh filename="package://description_robot/models/ackermann_rover/cubepilot/cubepilot.stl" scale="0.001 0.001 0.001"/>
+          <!-- <box size="${board_x} ${board_y} ${board_z}"/> -->
         </geometry>
         <material name="cubepilot_gray">
