Commit message: feat: scale meshes to match URDF geometry and bridge joint states for PX4 mode\n\n- Add mesh reference properties (mesh_wheelbase, mesh_separation,\n  mesh_wheel_diameter, mesh_base_rear_y) from donkey SDF\n- Scale chassis and wheel meshes to match wheel_base=0.174,\n  wheel_separation=0.174, wheel_diameter=0.077\n- Update collision cylinder radii to ${wheel_diameter/2}\n- Update controller wheel radii to 0.0385\n- Remove invalid <ros><namespace> from JointStatePublisher plugin\n- Add conditional parameter_bridge for /joint_states in PX4 SITL mode\n- Add --build/--build-only options to start_ros2_nodes.sh\n- Update architecture docs with build examples"

File: src/description_robot/models/ackermann_rover/ackermann_rover.urdf (robot description, URDF)
Before this commit: robot ackermann, 8 links, 7 joints
Links:
- link $(arg ns)/base_link: geometry collision box size=.3 .09 .12; visual mesh filename=package://description_robot/models/donkey/meshes/BaseReduce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 scale=${wheel_separation/mesh_separation} ${wheel_base/mesh_wheel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
- link $(arg ns)/front_left_wheel_link: geometry collision cylinder length=0.03 radius=${wheel_diameter/2}; visual mesh filename=package://description_robot/models/donkey/meshes/Wheel.dae scale=${wheel_diameter/mesh_wheel_diameter} 1 ${wheel_diameter/me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
- link $(arg ns)/front_right_wheel_link: geometry collision cylinder length=0.03 radius=${wheel_diameter/2}; visual mesh filename=package://description_robot/models/donkey/meshes/Wheel.dae scale=${wheel_diameter/mesh_wheel_diameter} 1 ${wheel_diameter/me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
- link $(arg ns)/rear_left_wheel_link: geometry collision cylinder length=0.03 radius=${wheel_diameter/2}; visual mesh filename=package://description_robot/models/donkey/meshes/Wheel.dae scale=${wheel_diameter/mesh_wheel_diameter} 1 ${wheel_diameter/me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
- link $(arg ns)/rear_right_wheel_link: geometry collision cylinder length=0.03 radius=${wheel_diameter/2}; visual mesh filename=package://description_robot/models/donkey/meshes/Wheel.dae scale=${wheel_diameter/mesh_wheel_diameter} 1 ${wheel_diameter/me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
