Commit message: fix(hw): Jetson hardware session fixes — realsense2_description removal, EKF tuning, telemetry broker
- docker/docker-compose.yml: add version: '2.3' for docker-compose v1.25 compatibility on Jetson host
- scripts/start_ros2_nodes.sh: disable RViz by default in --hw mode (NvRmMem GPU access denied in Docker)
- scripts/start_jetson_session.sh: pass broker_host arg to monitor.launch.py when --with-telemetry
- src/description_robot: replace all realsense2_description external package refs with local files
  - _d435.urdf.xacro, _d435i.urdf.xacro, _l515.urdf.xacro: use $(find description_robot)/... paths
  - Add urdf/_materials.urdf.xacro and urdf/_usb_plug.urdf.xacro (local copies)
  - gazebo_bringup.launch.py: remove realsense2_description from resource_roots
  - package.xml: remove exec_depend on realsense2_description
- src/rover_monitor/launch/monitor.launch.py: add broker_host launch arg, pass as param override
- src/rover_monitor/config/publisher.yaml: reset broker_host to localhost (dev default)
- src/rtabmap_bringup/launch/rtabmap_slam.launch.py: lower EKF frequency 30→15 Hz (Jetson ARM limit)

Co-Authored-By: Claude Sonnet 4.6 <noreply@anthropic.com>

File: src/description_robot/models/ackermann_rover/realsense/_d435.urdf.xacro (robot description, xacro)
@@ -8,6 +8,6 @@
 <robot name="sensor_d435" xmlns:xacro="http://ros.org/wiki/xacro">
   <!-- Includes -->
-  <xacro:include filename="$(find realsense2_description)/urdf/_materials.urdf.xacro" />
-  <xacro:include filename="$(find realsense2_description)/urdf/_usb_plug.urdf.xacro" />
+  <xacro:include filename="$(find description_robot)/models/ackermann_rover/realsense/urdf/_materials.urdf.xacro" />
+  <xacro:include filename="$(find description_robot)/models/ackermann_rover/realsense/urdf/_usb_plug.urdf.xacro" />
   <xacro:macro name="sensor_d435" params="parent *origin name:=camera use_nominal_extrinsics:=false add_plug:=false use_mesh:=true">
     <xacro:property name="M_PI" value="3.1415926535897931" />
@@ -53,5 +53,5 @@
           <origin xyz="${d435_zero_depth_to_glass + d435_glass_to_front} ${-d435_cam_depth_py} 0" rpy="${M_PI/2} 0 ${M_PI/2}"/>
           <geometry>
-            <mesh filename="package://realsense2_description/meshes/d435.dae" />
+            <mesh filename="package://description_robot/models/ackermann_rover/realsense/meshes/d435.dae" />
           </geometry>
         </xacro:if>

File: src/description_robot/models/ackermann_rover/realsense/_d435i.urdf.xacro (robot description, xacro)
@@ -7,5 +7,5 @@
 -->
 <robot name="sensor_d435i" xmlns:xacro="http://ros.org/wiki/xacro">
-  <xacro:include filename="$(find realsense2_description)/urdf/_d435.urdf.xacro"/>
+  <xacro:include filename="$(find description_robot)/models/ackermann_rover/realsense/_d435.urdf.xacro"/>
   <xacro:include filename="$(find description_robot)/models/ackermann_rover/realsense/_d435i_imu_modules.urdf.xacro"/>
   <xacro:include filename="$(find description_robot)/models/ackermann_rover/realsense/_d435i_sensors.urdf.xacro"/>

File: src/description_robot/models/ackermann_rover/realsense/_l515.urdf.xacro (robot description, xacro)
@@ -8,6 +8,6 @@
 <robot name="sensor_l515" xmlns:xacro="http://ros.org/wiki/xacro">
   <!-- Includes -->
-  <xacro:include filename="$(find realsense2_description)/urdf/_materials.urdf.xacro" />
-  <xacro:include filename="$(find realsense2_description)/urdf/_usb_plug.urdf.xacro" /> <!-- this specific plug does not apply to L515 -->
+  <xacro:include filename="$(find description_robot)/models/ackermann_rover/realsense/urdf/_materials.urdf.xacro" />
+  <xacro:include filename="$(find description_robot)/models/ackermann_rover/realsense/urdf/_usb_plug.urdf.xacro" /> <!-- this specific plug does not apply to L515 -->
   <xacro:include filename="$(find description_robot)/models/ackermann_rover/realsense/_l515_sensors.urdf.xacro"/>
   <xacro:macro name="sensor_l515" params="parent *origin name:=camera use_nominal_extrinsics:=false add_plug:=false use_mesh:=true add_sensors:=true">
